File: smarthome_v0.1.kicad_sch (KiCad schematic)
At the start: 67 parts, among them J1 USB_C_Receptacle_USB2.0_16P, J2 Screw_Terminal_01x06, J3 Screw_Terminal_01x06, J4 Conn_01x04_Pin, K1 HF46F_005-HS1, K2 HF46F_005-HS1, K3 HF46F_005-HS1, K4 HF46F_005-HS1, Q1 SS8050, Q2 SS8050, SW1 SW_Push, SW2 SW_Push, SW3 SW_Push, SW4 SW_Push, SW5 SW_Push, U1 ULN2003A, U2 CH340C, U3 AMS1117-3.3, U4 ESP32-WROOM-32

Commit message: revert PCB and schematic to original design, update BOM and firmware docs
Parts:
- removed SW3, SW4, SW5: SW_Push, Button_Switch_SMD:SW_Push_SPST_NO_Alps_SKRK, symbol Switch:SW_Push

Commit message: add navigation switches SW3, SW4, SW5 symbols to schematic
Parts:
- added SW3, SW4, SW5: SW_Push, Button_Switch_SMD:SW_Push_SPST_NO_Alps_SKRK, symbol Switch:SW_Push
Connections:
- net SWITCH_1/IO13: now also SW3.1
- net SWITCH_2/IO12: now also SW4.1
- net SWITCH_3/IO27: now also SW5.1
